Commit message: Convert MIT push shapes to URDF, loading/visualization of groundtruth trajectories in TDS

File: data/mit-push/obj/butter.urdf (robot description, URDF)
Before this commit: robot push_object, 1 links, 0 joints
Links:
- removed link baseLink
- added link link_object, mass 10.0; collision sphere radius=0.0065; collision sphere radius=0.0065
- added link link_x, mass 0
- added link link_y, mass 0
- added link link_yaw, mass 0
- added link link_z, mass 0
Joints:
- added joint joint_x: type prismatic, parent link_x, child link_y, origin xyz=0.0 0.0 0, axis 1 0 0, limit lower=-15 upper=15 effort=1000.0 velocity=5
- added joint joint_y: type prismatic, parent link_y, child link_z, origin xyz=0.0 0.0 0, axis 0 1 0, limit lower=-15 upper=15 effort=1000.0 velocity=5
- added joint joint_yaw: type continuous, parent link_yaw, child link_object, origin xyz=0.0 0.0 0, axis 0 0 1
- added joint joint_z: type prismatic, parent link_z, child link_yaw, origin xyz=0.0 0.0 0, axis 0 0 1, limit lower=-15 upper=15 effort=1000.0 velocity=5

File: data/mit-push/obj/ellip1.urdf (robot description, URDF)
Before this commit: robot push_object, 1 links, 0 joints
Links:
- removed link baseLink
- added link link_object, mass 10.0; collision sphere radius=0.0065; collision sphere radius=0.0065
- added link link_x, mass 0
- added link link_y, mass 0
- added link link_yaw, mass 0
- added link link_z, mass 0
Joints:
- added joint joint_x: type prismatic, parent link_x, child link_y, origin xyz=0.0 0.0 0, axis 1 0 0, limit lower=-15 upper=15 effort=1000.0 velocity=5
- added joint joint_y: type prismatic, parent link_y, child link_z, origin xyz=0.0 0.0 0, axis 0 1 0, limit lower=-15 upper=15 effort=1000.0 velocity=5
- added joint joint_yaw: type continuous, parent link_yaw, child link_object, origin xyz=0.0 0.0 0, axis 0 0 1
- added joint joint_z: type prismatic, parent link_z, child link_yaw, origin xyz=0.0 0.0 0, axis 0 0 1, limit lower=-15 upper=15 effort=1000.0 velocity=5

File: data/mit-push/obj/ellip2.urdf (robot description, URDF)
Before this commit: robot push_object, 1 links, 0 joints
Links:
- removed link baseLink
- added link link_object, mass 10.0; collision sphere radius=0.0065; collision sphere radius=0.0065
- added link link_x, mass 0
- added link link_y, mass 0
- added link link_yaw, mass 0
- added link link_z, mass 0
Joints:
- added joint joint_x: type prismatic, parent link_x, child link_y, origin xyz=0.0 0.0 0, axis 1 0 0, limit lower=-15 upper=15 effort=1000.0 velocity=5
- added joint joint_y: type prismatic, parent link_y, child link_z, origin xyz=0.0 0.0 0, axis 0 1 0, limit lower=-15 upper=15 effort=1000.0 velocity=5
- added joint joint_yaw: type continuous, parent link_yaw, child link_object, origin xyz=0.0 0.0 0, axis 0 0 1
- added joint joint_z: type prismatic, parent link_z, child link_yaw, origin xyz=0.0 0.0 0, axis 0 0 1, limit lower=-15 upper=15 effort=1000.0 velocity=5

File: data/mit-push/obj/ellip3.urdf (robot description, URDF)
Before this commit: robot push_object, 1 links, 0 joints
Links:
- removed link baseLink
- added link link_object, mass 10.0; collision sphere radius=0.0065; collision sphere radius=0.0065
- added link link_x, mass 0
- added link link_y, mass 0
- added link link_yaw, mass 0
- added link link_z, mass 0
Joints:
- added joint joint_x: type prismatic, parent link_x, child link_y, origin xyz=0.0 0.0 0, axis 1 0 0, limit lower=-15 upper=15 effort=1000.0 velocity=5
- added joint joint_y: type prismatic, parent link_y, child link_z, origin xyz=0.0 0.0 0, axis 0 1 0, limit lower=-15 upper=15 effort=1000.0 velocity=5
- added joint joint_yaw: type continuous, parent link_yaw, child link_object, origin xyz=0.0 0.0 0, axis 0 0 1
- added joint joint_z: type prismatic, parent link_z, child link_yaw, origin xyz=0.0 0.0 0, axis 0 0 1, limit lower=-15 upper=15 effort=1000.0 velocity=5

File: data/mit-push/obj/hex.urdf (robot description, URDF)
Before this commit: robot push_object, 1 links, 0 joints
Links:
- removed link baseLink
- added link link_object, mass 10.0; collision sphere radius=0.0065; collision sphere radius=0.0065
- added link link_x, mass 0
- added link link_y, mass 0
- added link link_yaw, mass 0
- added link link_z, mass 0
Joints:
- added joint joint_x: type prismatic, parent link_x, child link_y, origin xyz=0.0 0.0 0, axis 1 0 0, limit lower=-15 upper=15 effort=1000.0 velocity=5
- added joint joint_y: type prismatic, parent link_y, child link_z, origin xyz=0.0 0.0 0, axis 0 1 0, limit lower=-15 upper=15 effort=1000.0 velocity=5
- added joint joint_yaw: type continuous, parent link_yaw, child link_object, origin xyz=0.0 0.0 0, axis 0 0 1
- added joint joint_z: type prismatic, parent link_z, child link_yaw, origin xyz=0.0 0.0 0, axis 0 0 1, limit lower=-15 upper=15 effort=1000.0 velocity=5

File: data/mit-push/obj/rect1.urdf (robot description, URDF)
Before this commit: robot push_object, 1 links, 0 joints
Links:
- removed link baseLink
- added link link_object, mass 10.0; collision sphere radius=0.0065; collision sphere radius=0.0065
- added link link_x, mass 0
- added link link_y, mass 0
- added link link_yaw, mass 0
- added link link_z, mass 0
Joints:
- added joint joint_x: type prismatic, parent link_x, child link_y, origin xyz=0.0 0.0 0, axis 1 0 0, limit lower=-15 upper=15 effort=1000.0 velocity=5
- added joint joint_y: type prismatic, parent link_y, child link_z, origin xyz=0.0 0.0 0, axis 0 1 0, limit lower=-15 upper=15 effort=1000.0 velocity=5
- added joint joint_yaw: type continuous, parent link_yaw, child link_object, origin xyz=0.0 0.0 0, axis 0 0 1
- added joint joint_z: type prismatic, parent link_z, child link_yaw, origin xyz=0.0 0.0 0, axis 0 0 1, limit lower=-15 upper=15 effort=1000.0 velocity=5

File: data/mit-push/obj/rect2.urdf (robot description, URDF)
Before this commit: robot push_object, 1 links, 0 joints
Links:
- removed link baseLink
- added link link_object, mass 10.0; collision sphere radius=0.0065; collision sphere radius=0.0065
- added link link_x, mass 0
- added link link_y, mass 0
- added link link_yaw, mass 0
- added link link_z, mass 0
Joints:
- added joint joint_x: type prismatic, parent link_x, child link_y, origin xyz=0.0 0.0 0, axis 1 0 0, limit lower=-15 upper=15 effort=1000.0 velocity=5
- added joint joint_y: type prismatic, parent link_y, child link_z, origin xyz=0.0 0.0 0, axis 0 1 0, limit lower=-15 upper=15 effort=1000.0 velocity=5
- added joint joint_yaw: type continuous, parent link_yaw, child link_object, origin xyz=0.0 0.0 0, axis 0 0 1
- added joint joint_z: type prismatic, parent link_z, child link_yaw, origin xyz=0.0 0.0 0, axis 0 0 1, limit lower=-15 upper=15 effort=1000.0 velocity=5

File: data/mit-push/obj/rect3.urdf (robot description, URDF)
Before this commit: robot push_object, 1 links, 0 joints
Links:
- removed link baseLink
- added link link_object, mass 10.0; collision sphere radius=0.0065; collision sphere radius=0.0065
- added link link_x, mass 0
- added link link_y, mass 0
- added link link_yaw, mass 0
- added link link_z, mass 0
Joints:
- added joint joint_x: type prismatic, parent link_x, child link_y, origin xyz=0.0 0.0 0, axis 1 0 0, limit lower=-15 upper=15 effort=1000.0 velocity=5
- added joint joint_y: type prismatic, parent link_y, child link_z, origin xyz=0.0 0.0 0, axis 0 1 0, limit lower=-15 upper=15 effort=1000.0 velocity=5
- added joint joint_yaw: type continuous, parent link_yaw, child link_object, origin xyz=0.0 0.0 0, axis 0 0 1
- added joint joint_z: type prismatic, parent link_z, child link_yaw, origin xyz=0.0 0.0 0, axis 0 0 1, limit lower=-15 upper=15 effort=1000.0 velocity=5

File: data/mit-push/obj/tri1.urdf (robot description, URDF)
Before this commit: robot push_object, 1 links, 0 joints
Links:
- removed link baseLink
- added link link_object, mass 10.0; collision sphere radius=0.0065; collision sphere radius=0.0065
- added link link_x, mass 0
- added link link_y, mass 0
- added link link_yaw, mass 0
- added link link_z, mass 0
Joints:
- added joint joint_x: type prismatic, parent link_x, child link_y, origin xyz=0.0 0.0 0, axis 1 0 0, limit lower=-15 upper=15 effort=1000.0 velocity=5
- added joint joint_y: type prismatic, parent link_y, child link_z, origin xyz=0.0 0.0 0, axis 0 1 0, limit lower=-15 upper=15 effort=1000.0 velocity=5
- added joint joint_yaw: type continuous, parent link_yaw, child link_object, origin xyz=0.0 0.0 0, axis 0 0 1
- added joint joint_z: type prismatic, parent link_z, child link_yaw, origin xyz=0.0 0.0 0, axis 0 0 1, limit lower=-15 upper=15 effort=1000.0 velocity=5

File: data/mit-push/obj/tri2.urdf (robot description, URDF)
Before this commit: robot push_object, 1 links, 0 joints
Links:
- removed link baseLink
- added link link_object, mass 10.0; collision sphere radius=0.0065; collision sphere radius=0.0065
- added link link_x, mass 0
- added link link_y, mass 0
- added link link_yaw, mass 0
- added link link_z, mass 0
Joints:
- added joint joint_x: type prismatic, parent link_x, child link_y, origin xyz=0.0 0.0 0, axis 1 0 0, limit lower=-15 upper=15 effort=1000.0 velocity=5
- added joint joint_y: type prismatic, parent link_y, child link_z, origin xyz=0.0 0.0 0, axis 0 1 0, limit lower=-15 upper=15 effort=1000.0 velocity=5
- added joint joint_yaw: type continuous, parent link_yaw, child link_object, origin xyz=0.0 0.0 0, axis 0 0 1
- added joint joint_z: type prismatic, parent link_z, child link_yaw, origin xyz=0.0 0.0 0, axis 0 0 1, limit lower=-15 upper=15 effort=1000.0 velocity=5

File: data/mit-push/obj/tri3.urdf (robot description, URDF)
Before this commit: robot push_object, 1 links, 0 joints
Links:
- removed link baseLink
- added link link_object, mass 10.0; collision sphere radius=0.0065; collision sphere radius=0.0065
- added link link_x, mass 0
- added link link_y, mass 0
- added link link_yaw, mass 0
- added link link_z, mass 0
Joints:
- added joint joint_x: type prismatic, parent link_x, child link_y, origin xyz=0.0 0.0 0, axis 1 0 0, limit lower=-15 upper=15 effort=1000.0 velocity=5
- added joint joint_y: type prismatic, parent link_y, child link_z, origin xyz=0.0 0.0 0, axis 0 1 0, limit lower=-15 upper=15 effort=1000.0 velocity=5
- added joint joint_yaw: type continuous, parent link_yaw, child link_object, origin xyz=0.0 0.0 0, axis 0 0 1
- added joint joint_z: type prismatic, parent link_z, child link_yaw, origin xyz=0.0 0.0 0, axis 0 0 1, limit lower=-15 upper=15 effort=1000.0 velocity=5

Commit message: Correct yaw angle of pushed object

File: data/mit-push/obj/butter.urdf (robot description, URDF)
Before this commit: robot push_object, 5 links, 4 joints
Links:
- link link_object: mass 10.0 -> 0.006350

File: data/mit-push/obj/ellip1.urdf (robot description, URDF)
Before this commit: robot push_object, 5 links, 4 joints
Links:
- link link_object: mass 10.0 -> 0.006350

File: data/mit-push/obj/ellip2.urdf (robot description, URDF)
Before this commit: robot push_object, 5 links, 4 joints
Links:
- link link_object: mass 10.0 -> 0.006350

File: data/mit-push/obj/ellip3.urdf (robot description, URDF)
Before this commit: robot push_object, 5 links, 4 joints
Links:
- link link_object: mass 10.0 -> 0.006350

File: data/mit-push/obj/hex.urdf (robot description, URDF)
Before this commit: robot push_object, 5 links, 4 joints
Links:
- link link_object: mass 10.0 -> 0.006350

File: data/mit-push/obj/rect1.urdf (robot description, URDF)
Before this commit: robot push_object, 5 links, 4 joints
Links:
- link link_object: mass 0.1 -> 0.006350

File: data/mit-push/obj/rect2.urdf (robot description, URDF)
Before this commit: robot push_object, 5 links, 4 joints
Links:
- link link_object: mass 10.0 -> 0.006350

File: data/mit-push/obj/rect3.urdf (robot description, URDF)
Before this commit: robot push_object, 5 links, 4 joints
Links:
- link link_object: mass 10.0 -> 0.006350

File: data/mit-push/obj/tri1.urdf (robot description, URDF)
Before this commit: robot push_object, 5 links, 4 joints
Links:
- link link_object: mass 10.0 -> 0.006350

File: data/mit-push/obj/tri2.urdf (robot description, URDF)
Before this commit: robot push_object, 5 links, 4 joints
Links:
- link link_object: mass 10.0 -> 0.006350

File: data/mit-push/obj/tri3.urdf (robot description, URDF)
Before this commit: robot push_object, 5 links, 4 joints
Links:
- link link_object: mass 10.0 -> 0.006350

Commit message: Improve neural scalar, push experiment

File: data/mit-push/obj/butter.urdf (robot description, URDF)
Before this commit: robot push_object, 5 links, 4 joints
Links:
- link link_object: geometry collision sphere radius=0.0065; collision sphere radius=0.0065

File: data/mit-push/obj/ellip1.urdf (robot description, URDF)
Before this commit: robot push_object, 5 links, 4 joints
Links:
- link link_object: geometry collision sphere radius=0.0065; collision sphere radius=0.0065

File: data/mit-push/obj/ellip2.urdf (robot description, URDF)
Before this commit: robot push_object, 5 links, 4 joints
Links:
- link link_object: geometry collision sphere radius=0.0065; collision sphere radius=0.0065

File: data/mit-push/obj/ellip3.urdf (robot description, URDF)
Before this commit: robot push_object, 5 links, 4 joints
Links:
- link link_object: geometry collision sphere radius=0.0065; collision sphere radius=0.0065

File: data/mit-push/obj/hex.urdf (robot description, URDF)
Before this commit: robot push_object, 5 links, 4 joints
Links:
- link link_object: geometry collision sphere radius=0.0065; collision sphere radius=0.0065

File: data/mit-push/obj/rect1.urdf (robot description, URDF)
Before this commit: robot push_object, 5 links, 4 joints
Links:
- link link_object: geometry collision sphere radius=0.0065; collision sphere radius=0.0065

File: data/mit-push/obj/rect2.urdf (robot description, URDF)
Before this commit: robot push_object, 5 links, 4 joints
Links:
- link link_object: geometry collision sphere radius=0.0065; collision sphere radius=0.0065

File: data/mit-push/obj/rect3.urdf (robot description, URDF)
Before this commit: robot push_object, 5 links, 4 joints
Links:
- link link_object: geometry collision sphere radius=0.0065; collision sphere radius=0.0065

File: data/mit-push/obj/tri1.urdf (robot description, URDF)
Before this commit: robot push_object, 5 links, 4 joints
Links:
- link link_object: geometry collision sphere radius=0.0065; collision sphere radius=0.0065

File: data/mit-push/obj/tri2.urdf (robot description, URDF)
Before this commit: robot push_object, 5 links, 4 joints
Links:
- link link_object: geometry collision sphere radius=0.0065; collision sphere radius=0.0065

File: data/mit-push/obj/tri3.urdf (robot description, URDF)
Before this commit: robot push_object, 5 links, 4 joints
Links:
- link link_object: geometry collision sphere radius=0.0065; collision sphere radius=0.0065
