Commit message: Split masses, add visualization tools

File: data/swimmer/swimmer03/swimmer03.urdf (robot description, URDF)
Before this commit: robot swimmer03, 6 links, 5 joints
Links:
- link link00: mass 0.01 -> 0.0033333333333333335
- link xslide: mass 0 -> 0.0033333333333333335
- link yslide: mass 0 -> 0.0033333333333333335

File: data/swimmer/swimmer04/swimmer04.urdf (robot description, URDF)
Before this commit: robot swimmer04, 7 links, 6 joints
Links:
- link link00: mass 0.01 -> 0.0033333333333333335
- link xslide: mass 0 -> 0.0033333333333333335
- link yslide: mass 0 -> 0.0033333333333333335

File: data/swimmer/swimmer05/swimmer05.urdf (robot description, URDF)
Before this commit: robot swimmer05, 8 links, 7 joints
Links:
- link link00: mass 0.01 -> 0.0033333333333333335
- link xslide: mass 0 -> 0.0033333333333333335
- link yslide: mass 0 -> 0.0033333333333333335

File: data/swimmer/swimmer06/swimmer06.urdf (robot description, URDF)
Before this commit: robot swimmer06, 9 links, 8 joints
Links:
- link link00: mass 0.01 -> 0.0033333333333333335
- link xslide: mass 0 -> 0.0033333333333333335
- link yslide: mass 0 -> 0.0033333333333333335

File: data/swimmer/swimmer07/swimmer07.urdf (robot description, URDF)
Before this commit: robot swimmer07, 10 links, 9 joints
Links:
- link link00: mass 0.01 -> 0.0033333333333333335
- link xslide: mass 0 -> 0.0033333333333333335
- link yslide: mass 0 -> 0.0033333333333333335

File: data/swimmer/swimmer08/swimmer08.urdf (robot description, URDF)
Before this commit: robot swimmer08, 11 links, 10 joints
Links:
- link link00: mass 0.01 -> 0.0033333333333333335
- link xslide: mass 0 -> 0.0033333333333333335
- link yslide: mass 0 -> 0.0033333333333333335

File: data/swimmer/swimmer09/swimmer09.urdf (robot description, URDF)
Before this commit: robot swimmer09, 12 links, 11 joints
Links:
- link link00: mass 0.01 -> 0.0033333333333333335
- link xslide: mass 0 -> 0.0033333333333333335
- link yslide: mass 0 -> 0.0033333333333333335

File: data/swimmer/swimmer10/swimmer10.urdf (robot description, URDF)
Before this commit: robot swimmer10, 13 links, 12 joints
Links:
- link link00: mass 0.01 -> 0.0033333333333333335
- link xslide: mass 0 -> 0.0033333333333333335
- link yslide: mass 0 -> 0.0033333333333333335

File: data/swimmer/swimmer11/swimmer11.urdf (robot description, URDF)
Before this commit: robot swimmer11, 14 links, 13 joints
Links:
- link link00: mass 0.01 -> 0.0033333333333333335
- link xslide: mass 0 -> 0.0033333333333333335
- link yslide: mass 0 -> 0.0033333333333333335

File: data/swimmer/swimmer12/swimmer12.urdf (robot description, URDF)
Before this commit: robot swimmer12, 15 links, 14 joints
Links:
- link link00: mass 0.01 -> 0.0033333333333333335
- link xslide: mass 0 -> 0.0033333333333333335
- link yslide: mass 0 -> 0.0033333333333333335

File: data/swimmer/swimmer13/swimmer13.urdf (robot description, URDF)
Before this commit: robot swimmer13, 16 links, 15 joints
Links:
- link link00: mass 0.01 -> 0.0033333333333333335
- link xslide: mass 0 -> 0.0033333333333333335
- link yslide: mass 0 -> 0.0033333333333333335

File: data/swimmer/swimmer14/swimmer14.urdf (robot description, URDF)
Before this commit: robot swimmer14, 17 links, 16 joints
Links:
- link link00: mass 0.01 -> 0.0033333333333333335
- link xslide: mass 0 -> 0.0033333333333333335
- link yslide: mass 0 -> 0.0033333333333333335
